File: proyectos/proyectos.sch (KiCad schematic (older format))
At the start: 58 parts, among them P1 CONN_01X02, P2 CONN_01X03, P3 CONN_01X05, P4 CONN_01X03, P5 CONN_01X03, P6 CONN_01X02, P7 CONN_01X01, P8 CONN_01X01, U1 AD8232_A, U2 ADP3334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

Commit message: version 1.9 ECG Y PIC
nuevo cambio de regulador  y logo
Parts:
- removed C9: 0.1uF, Capacitors_SMD:C_0805_HandSoldering, symbol 0.1uF
- added C9: 1nF_1208, Capacitors_SMD:C_1206_HandSoldering, symbol 1nF_1208
Connections:
- net +5V: no longer U2.2 (SD)
- net +vs: now also C9.1
- net GND: now also U2.2 (SD)
- net at R16.2, R17.1, U2.7 (FB): now also C9.2
Changed lines of the file:
@@
 Connection ~ 2100 7150
-Wire Wire Line
-	8800 1300 8800 1700
-Wire Wire Line
-	8800 1700 8900 1700
 Wire Wire Line
 	8550 1750 8550 2000
@@
 	0    1    1    0
 $EndComp
-$Comp
-L ADP3334 U2
-U 1 1 591DA311
-P 9500 1500
-F 0 "U2" H 9650 750 60  0000 C CNN
-F 1 "ADP3334" H 9500 1700 60  0000 C CNN
-F 2 "Housings_SOIC:SOIC-8_3.9x4.9mm_Pitch1.27mm" H 9800 2000 60  0001 C CNN
-F 3 "" H 9400 1500 60  0000 C CNN
-F 4 "ADP3334ARZ" H 9750 850 60  0001 C CNN "Adjustable Low Dropout Regulator "
-	1    9500 1500
-	1    0    0    -1
-$EndComp
 Wire Wire Line
 	8900 1300 8800 1300
@@
 	10150 1700 10150 1750
 Wire Wire Line
-	10150 1950 10150 2050
-Wire Wire Line
-	10150 2050 9500 2050
+	10150 2050 10150 1950
+Wire Wire Line
+	8800 2050 10150 2050
 Connection ~ 9500 2050
 $Comp
@@
 	1    0    0    -1
 $EndComp
-$Comp
-L 0.1uF C9
-U 1 1 591E6691
-P 10450 1600
-F 0 "C9" H 10460 1670 50  0000 L CNN
-F 1 "0.1uF" H 10460 1520 50  0000 L CNN
-F 2 "Capacitors_SMD:C_0805_HandSoldering" H 10360 1570 50  0001 C CNN
-F 3 "" H 10460 1670 50  0000 C CNN
-F 4 "1276-2450-2-ND" H 10560 1770 60  0001 C CNN "CAP CER 0.1UF 25V X7R 0805"
-	1    10450 1600
-	1    0    0    -1
-$EndComp
 Connection ~ 10450 1500
 Connection ~ 10150 1700
@@
 Wire Wire Line
 	10650 2050 10650 1750
+$Comp
+L 1nF_1208 C9
+U 1 1 591E0EF5
+P 10450 1600
+F 0 "C9" H 10460 1670 50  0000 L CNN
+F 1 "1nF_1208" H 10460 1520 50  0000 L CNN
+F 2 "Capacitors_SMD:C_1206_HandSoldering" H 10360 1570 50  0001 C CNN
+F 3 "" H 10460 1670 50  0000 C CNN
+F 4 "1276-1050-2-ND" H 10560 1770 60  0001 C CNN "CAP CER 1000PF 50V X7R 1206"
+	1    10450 1600
+	1    0    0    -1
+$EndComp
+Wire Wire Line
+	8800 1300 8800 1500
+$Comp
+L ADP3334 U2
+U 1 1 591E1D97
+P 9500 1500
+F 0 "U2" H 9650 750 60  0000 C CNN
+F 1 "ADP3334" H 9500 1750 60  0000 C CNN
+F 2 "Housings_SOIC:SOIC-8_3.9x4.9mm_Pitch1.27mm" H 9800 2000 60  0001 C CNN
+F 3 "" H 9400 1500 60  0000 C CNN
+F 4 "ADP3334ARZ" H 9750 850 60  0001 C CNN "Adjustable Low Dropout Regulator "
+	1    9500 1500
+	1    0    0    -1
+$EndComp
+Wire Wire Line
+	8900 1700 8800 1700
+Wire Wire Line
+	8800 1700 8800 2050
 $EndSCHEMATC

Commit message: version 2.0 ecg y pic
archivo para panelizar
Parts:
- removed P7, P8: CONN_01X01, Huellas:MountingHole_1.8mm_Pad, symbol CONN_01X01
Connections:
- no-connect marks 2 -> 0
Changed lines of the file:
@@
 $EndComp
-$Comp
-L CONN_01X01 P8
-U 1 1 591B656B
-P 10300 5900
-F 0 "P8" H 10300 6000 50  0000 C CNN
-F 1 "CONN_01X01" V 10400 5900 50  0000 C CNN
-F 2 "Huellas:MountingHole_1.8mm_Pad" H 10300 5900 50  0001 C CNN
-F 3 "" H 10300 5900 50  0000 C CNN
-	1    10300 5900
-	1    0    0    -1
-$EndComp
-$Comp
-L CONN_01X01 P7
-U 1 1 591B6624
-P 9350 5900
-F 0 "P7" H 9350 6000 50  0000 C CNN
-F 1 "CONN_01X01" V 9450 5900 50  0000 C CNN
-F 2 "Huellas:MountingHole_1.8mm_Pad" H 9350 5900 50  0001 C CNN
-F 3 "" H 9350 5900 50  0000 C CNN
-	1    9350 5900
-	1    0    0    -1
-$EndComp
-NoConn ~ 10100 5900
-NoConn ~ 9150 5900
 $Comp
 L 22pF C11
